File: Choc/THT/main.kicad_pcb (KiCad board)
At the start: 2 copper layers, 123.4 x 89.9 mm, 74 parts

Commit message: Add mount holes
Parts:
- removed the BQ24075 at (154.3, 115.5)
- removed the CAP at (244.2, 115.7)
- removed the CAP at (153.6, 118.0)
- removed the CAP at (157.3, 113.9)
- removed the CAP at (150.1, 117.0)
- removed the LED at (150.6, 114.3)
- removed the LED at (244.2, 119.9)
- removed the RES at (125.0, 120.0)
- removed the RES at (155.6, 118.0)
- removed the RES at (150.1, 115.5)
- removed the RES at (155.6, 119.0)
- removed the RES at (244.2, 111.3)
- removed the RES at (127.2, 120.0)
- added RES: RES, Resistor_THT:R_Axial_DIN0204_L3.6mm_D1.6mm_P5.08mm_Horizontal, F.Cu at (104.7, 134.2)
Routing:
- net GND: track 619.8 -> 584.2 mm, vias 11 -> 9
- net VDDH: track 42.8 -> 22.3 mm
- net VBAT: track 10.1 -> 5.06 mm
- net VBUS: track 49.7 -> 45.1 mm
- net (no net): track 58.2 -> 56.0 mm
