File: Choc/SMD/main.kicad_pcb (KiCad board)
At the start: 2 copper layers, 128.7 x 89.9 mm, 66 parts

Commit message: Copper fill
Parts:
- removed the G*** at (403.5, 120.6)
- removed the G*** at (393.6, 118.5)
- removed the USB-C at (119.8, 136.9)
- added 0: MountingHole_3.2mm_M3_Pad_Via, MountingHole:MountingHole_3.2mm_M3_Pad_Via, F.Cu at (155.5, 128.8)
- added ?: , clipboard:8583f098-8525-47d3-99c4-a63cf4c513a4, F.Cu at (121.9, 133.6)
- added GND: TestPoint_Plated_Hole_D2.0mm, TestPoint:TestPoint_Plated_Hole_D2.0mm, F.Cu at (168.2, 128.8)
- added RESET: SW_PTS526_SM08_SMTR2_LFS, PTS526_SM08_SMTR2_LFS:SW_PTS526_SM08_SMTR2_LFS, F.Cu at (162.3, 134.5)
- added SWDCLK: TestPoint_Plated_Hole_D2.0mm, TestPoint:TestPoint_Plated_Hole_D2.0mm, F.Cu at (146.4, 144.6)
- added SWDIO: TestPoint_Plated_Hole_D2.0mm, TestPoint:TestPoint_Plated_Hole_D2.0mm, F.Cu at (150.0, 144.6)
- added USB-C: MOLEX_2169900003, 2169900003:MOLEX_2169900003, F.Cu at (117.0, 137.9)
- added VBAT: TestPoint_Plated_Hole_D2.0mm, TestPoint:TestPoint_Plated_Hole_D2.0mm, F.Cu at (163.6, 128.8)
- moved RES 1.05 mm to (120.8, 129.3)
- moved S1 0.90 mm to (194.3, 143.8)
- moved S2 0.90 mm to (194.3, 143.8)
- renumbered REF** to 0
Connections:
- BQ24075 pad ISET: GND -> (no net)
- BQ24075 pad TS: GND -> (no net)
- RES pad 2: GND -> (no net) (x2)
- nRF52833 pad 1: (no net) -> GND
- nRF52833 pad 28: (no net) -> RESET
Routing:
- net GND: track 597.0 -> 29.6 mm, vias 5 -> 2
- net RESET: track 0.00 -> 29.3 mm, vias 0 -> 2
- net (no net): track 5.58 -> 27.4 mm
- net VBAT: track 5.06 -> 16.9 mm
- net D-: track 34.9 -> 46.1 mm, vias 2 -> 3
- net K21: track 9.57 -> 19.8 mm
- net D+: track 31.1 -> 38.7 mm
- net VBUS: track 46.8 -> 52.7 mm, vias 2 -> 3
- net K1: track 33.9 -> 37.4 mm
- net K2: track 54.6 -> 52.8 mm
- net K19: track 60.3 -> 59.4 mm
- net K3: track 55.8 -> 56.5 mm
- added copper zone on B.Cu, net GND
- added copper zone on F.Cu, net GND
Other:
- board size 128.7 x 89.9 mm -> 128 x 89.4 mm
- board text added: "Estoc V0.1 PotatoMasha"
