File: Choc/SMD/main.kicad_sch (KiCad schematic)
At the start: 33 parts, among them SW10 SW_DPST_x2, SW11 SW_DPST_x2, SW12 SW_DPST_x2, SW13 SW_DPST_x2, SW14 SW_DPST_x2, SW15 SW_DPST_x2, SW16 SW_DPST_x2, SW17 SW_DPST_x2, SW18 SW_DPST_x2, SW19 SW_DPST_x2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

Commit message: Copper fill
Parts:
- added S1: (no value), symbol PTS526_SM08_SMTR2_LFS:PTS526_SM08_SMTR2_LFS
- C1: value (none) -> 1uF
- C2, C3: value (none) -> 4.7uF
- D1: value (none) -> LED
- J1: value (none) -> USB_C_2.0
- R1, R2: value (none) -> 5.1kΩ
- R3: value (none) -> 2kΩ
- R4: value (none) -> 10kΩ
- SW1: value (none) -> SW_DPST_x2
- U2: value (none) -> BQ24075; footprint (none) -> Package_DFN_QFN:VQFN-16-1EP_3x3mm_P0.5mm_EP1.6x1.6mm
Connections:
- net GND: now also S1.3, S1.4
- net RESET: now reaches U1.28 (P0.18)
- net RESET: now also S1.1, S1.2
- no-connect marks 36 -> 35
Changed lines of the file:
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@@
   (no_connect (at 81.28 125.73))
   (no_connect (at 73.66 125.73))
-  (no_connect (at 66.04 125.73))
   (no_connect (at 243.84 157.48))
   (no_connect (at 220.98 165.1))
@@
     )
   )
+  (global_label "RESET" (shape input) (at 203.2 95.25 180) (fields_autoplaced)
+    (effects (font (size 1.27 1.27)) (justify right))
+    (property "Intersheet References" "${INTERSHEET_REFS}" (id 0) (at 195.0417 95.1706 0)
+      (effects (font (size 1.27 1.27)) (justify right) hide)
+    )
+  )
   (global_label "D+" (shape input) (at 36.83 106.68 180) (fields_autoplaced)
     (effects (font (size 1.27 1.27)) (justify right))
@@
     )
   )
+  (global_label "RESET" (shape input) (at 66.04 125.73 270) (fields_autoplaced)
+    (effects (font (size 1.27 1.27)) (justify right))
+    (property "Intersheet References" "${INTERSHEET_REFS}" (id 0) (at 65.9606 133.8883 90)
+      (effects (font (size 1.27 1.27)) (justify right) hide)
+    )
+  )
   (global_label "K14" (shape input) (at 36.83 99.06 180) (fields_autoplaced)
     (effects (font (size 1.27 1.27)) (justify right))
@@
       (effects (font (size 1.27 1.27)) (justify right))
     )
-    (property "Value" "" (id 1) (at 238.76 40.6399 0)
+    (property "Value" "4.7uF" (id 1) (at 238.76 40.6399 0)
       (effects (font (size 1.27 1.27)) (justify right))
     )
@@
     (in_bom yes) (on_board yes)
     (property "Reference" "R3" (id 0) (at 199.39 66.04 90))
-    (property "Value" "" (id 1) (at 199.39 68.58 90))
+    (property "Value" "2kΩ" (id 1) (at 199.39 68.58 90))
     (property "Footprint" "" (id 2) (at 199.39 65.278 90)
       (effects (font (size 1.27 1.27)) hide)
@@
     (in_bom yes) (on_board yes)
     (property "Reference" "SW1" (id 0) (at 25.4 162.56 0))
-    (property "Value" "" (id 1) (at 39.37 162.56 0))
+    (property "Value" "SW_DPST_x2" (id 1) (at 39.37 162.56 0))
     (property "Footprint" "" (id 2) (at 30.48 163.83 0)
       (effects (font (size 1.27 1.27)) hide)
@@
       (effects (font (size 1.27 1.27)) (justify left))
     )
-    (property "Value" "" (id 1) (at 217.9194 38.1 0)
+    (property "Value" "BQ24075" (id 1) (at 217.9194 38.1 0)
       (effects (font (size 1.27 1.27)) (justify left))
     )
-    (property "Footprint" "" (id 2) (at 223.52 67.31 0)
+    (property "Footprint" "Package_DFN_QFN:VQFN-16-1EP_3x3mm_P0.5mm_EP1.6x1.6mm" (id 2) (at 223.52 67.31 0)
       (effects (font (size 1.27 1.27)) (justify left) hide)
     )
@@
     (in_bom yes) (on_board yes)
     (property "Reference" "C1" (id 0) (at 212.09 29.21 90))
-    (property "Value" "" (id 1) (at 212.09 31.75 90))
+    (property "Value" "1uF" (id 1) (at 212.09 31.75 90))
     (property "Footprint" "" (id 2) (at 215.9 34.5948 0)
       (effects (font (size 1.27 1.27)) hide)
@@
     (in_bom yes) (on_board yes)
     (property "Reference" "R2" (id 0) (at 255.27 137.16 90))
-    (property "Value" "" (id 1) (at 255.27 139.7 90))
+    (property "Value" "5.1kΩ" (id 1) (at 255.27 139.7 90))
     (property "Footprint" "" (id 2) (at 255.27 136.398 90)
       (effects (font (size 1.27 1.27)) hide)
@@
     (in_bom yes) (on_board yes) (fields_autoplaced)
     (property "Reference" "J1" (id 0) (at 228.6 119.38 0))
-    (property "Value" "" (id 1) (at 228.6 121.92 0))
+    (property "Value" "USB_C_2.0" (id 1) (at 228.6 121.92 0))
     (property "Footprint" "" (id 2) (at 232.41 142.24 0)
       (effects (font (size 1.27 1.27)) hide)
@@
       (effects (font (size 1.27 1.27)) hide)
     )
-    (property "Value" "" (id 1) (at 228.6 168.91 0))
+    (property "Value" "GND" (id 1) (at 228.6 168.91 0))
     (property "Footprint" "" (id 2) (at 228.6 165.1 0)
       (effects (font (size 1.27 1.27)) hide)
@@
     (in_bom yes) (on_board yes)
     (property "Reference" "D1" (id 0) (at 233.68 68.58 0))
-    (property "Value" "" (id 1) (at 233.68 66.04 0))
+    (property "Value" "LED" (id 1) (at 233.68 66.04 0))
     (property "Footprint" "" (id 2) (at 232.41 63.5 0)
       (effects (font (size 1.27 1.27)) hide)
@@
     (in_bom yes) (on_board yes)
     (property "Reference" "R1" (id 0) (at 255.27 127 90))
-    (property "Value" "" (id 1) (at 255.27 129.54 90))
+    (property "Value" "5.1kΩ" (id 1) (at 255.27 129.54 90))
     (property "Footprint" "" (id 2) (at 255.27 133.858 90)
       (effects (font (size 1.27 1.27)) hide)
@@
     )
     (property "Datasheet" "" (id 3) (at 110.49 53.34 0)
+      (effects (font (size 1.27 1.27)) hide)
+    )
+    (pin "1")
+  )
+  (symbol (lib_id "power:GND") (at 218.44 95.25 90) (unit 1)
+    (in_bom yes) (on_board yes)
+    (property "Reference" "#PWR?" (id 0) (at 224.79 95.25 0)
+      (effects (font (size 1.27 1.27)) hide)
+    )
+    (property "Value" "GND" (id 1) (at 222.25 95.25 0))
+    (property "Footprint" "" (id 2) (at 218.44 95.25 0)
+      (effects (font (size 1.27 1.27)) hide)
+    )
+    (property "Datasheet" "" (id 3) (at 218.44 95.25 0)
       (effects (font (size 1.27 1.27)) hide)
     )
@@
     (in_bom yes) (on_board yes)
     (property "Reference" "R4" (id 0) (at 232.41 53.34 90))
-    (property "Value" "" (id 1) (at 232.41 58.42 90))
+    (property "Value" "10kΩ" (id 1) (at 232.41 58.42 90))
     (property "Footprint" "" (id 2) (at 232.41 57.658 90)
       (effects (font (size 1.27 1.27)) hide)
@@
     )
     (pin "1")
+  )
+  (symbol (lib_id "PTS526_SM08_SMTR2_LFS:PTS526_SM08_SMTR2_LFS") (at 210.82 95.25 0) (unit 1)
+    (in_bom yes) (on_board yes) (fields_autoplaced)
+    (property "Reference" "S1" (id 0) (at 210.82 87.63 0))
+    (property "Value" "" (id 1) (at 210.82 90.17 0))
+    (property "Footprint" "" (id 2) (at 210.82 95.25 0)
+      (effects (font (size 1.27 1.27)) (justify left bottom) hide)
+    )
+    (property "Datasheet" "" (id 3) (at 210.82 95.25 0)
+      (effects (font (size 1.27 1.27)) (justify left bottom) hide)
+    )
+    (property "MANUFACTURER" "C&K" (id 4) (at 210.82 95.25 0)
+      (effects (font (size 1.27 1.27)) (justify left bottom) hide)
+    )
+    (property "PARTREV" "20 mar 19" (id 5) (at 210.82 95.25 0)
+      (effects (font (size 1.27 1.27)) (justify left bottom) hide)
+    )
+    (property "MAXIMUM_PACKAGE_HEIGHT" "0.95mm" (id 6) (at 210.82 95.25 0)
+      (effects (font (size 1.27 1.27)) (justify left bottom) hide)
+    )
+    (property "STANDARD" "Manufacturer Recommendations" (id 7) (at 210.82 95.25 0)
+      (effects (font (size 1.27 1.27)) (justify left bottom) hide)
+    )
+    (pin "1")
+    (pin "2")
+    (pin "3")
+    (pin "4")
   )
   (symbol (lib_id "power:GND") (at 123.19 163.83 90) (unit 1)
@@
       (effects (font (size 1.27 1.27)) (justify right))
     )
-    (property "Value" "" (id 1) (at 251.46 55.88 0)
+    (property "Value" "4.7uF" (id 1) (at 251.46 55.88 0)
       (effects (font (size 1.27 1.27)) (justify right))
     )
@@
       (reference "#PWR0135") (unit 1) (value "GND") (footprint "")
     )
+    (path "/c0d3b680-12d3-4797-b22a-0bdc5b1b9f58"
+      (reference "#PWR?") (unit 1) (value "GND") (footprint "")
+    )
     (path "/37d25267-4a3f-4c6f-a26e-a466407b566b"
       (reference "C1") (unit 1) (value "1uF") (footprint "")
@@
       (reference "R5") (unit 1) (value "10kΩ") (footprint "")
     )
+    (path "/d8e0804c-9de4-4c91-936a-e3db1cda0edc"
+      (reference "S1") (unit 1) (value "PTS526_SM08_SMTR2_LFS") (footprint "SW_PTS526_SM08_SMTR2_LFS")
+    )
     (path "/2797e55b-ab07-4407-8f59-7c2f57176870"
