File: V0.2/main.kicad_pcb (KiCad board)
At the start: 2 copper layers, 127.5 x 87.9 mm, 72 parts

Commit message: Finalized design
Parts:
- removed the CAP at (205.5, 85.0)
- removed the CAP at (201.4, 81.2)
- removed the CAP at (213.3, 83.8)
- removed the CAP at (204.4, 88.2)
- removed G*** (x2): LOGO, LOGO
- removed the LED at (201.6, 87.9)
- removed the RES at (205.5, 82.8)
- removed the RES at (202.9, 88.2)
- removed the RES at (213.3, 85.5)
- removed the RES at (206.5, 82.8)
- added CAP: CAP, Capacitor_SMD:C_0402_1005Metric, F.Cu at (133.3, 89.8)
- added CAP: CAP, Capacitor_SMD:C_0402_1005Metric, F.Cu at (136.0, 92.1)
- added CAP: CAP, Capacitor_SMD:C_0402_1005Metric, F.Cu at (129.6, 94.4)
- added LED: LED, LED_SMD:LED_0603_1608Metric, F.Cu at (163.9, 133.3)
- added LED: LED, LED_SMD:LED_0603_1608Metric, F.Cu at (164.5, 129.4)
- added RES: RES, Resistor_SMD:R_0402_1005Metric, F.Cu at (162.7, 133.1)
- added RES: RES, Resistor_SMD:R_0402_1005Metric, F.Cu at (163.3, 129.2)
- added RES: RES, Resistor_SMD:R_0402_1005Metric, F.Cu at (131.2, 90.3)
- added RES: RES, Resistor_SMD:R_0402_1005Metric, F.Cu at (131.2, 89.3)
- added SWCLK: TestPoint_Keystone_5000-5004_Miniature, TestPoint:TestPoint_Keystone_5000-5004_Miniature, F.Cu at (161.1, 138.3)
- added SWIO: TestPoint_Keystone_5000-5004_Miniature, TestPoint:TestPoint_Keystone_5000-5004_Miniature, F.Cu at (164.4, 138.3)
- JST: renamed from REF**; value JST_BM02B-ACHSS-GAN-TF_LF__SN_ -> JST_BM02B
- RES (x2): renamed from REF**; value R_0603_1608Metric -> RES
- RES (x2): renamed from REF**; value C_0603_1608Metric -> C
- Y: renamed from REF**; value Crystal_SMD_MicroCrystal_CM9V-T1A-2Pin_1.6x1.0mm -> Y1
- moved BQ24075 70.8 mm to (132.6, 93.0), turned to 0 degrees
- moved SWITCH 36.0 mm to (125.3, 78.7)
- moved Button 13.3 mm to (165.1, 80.0)
- moved JST 0.20 mm to (143.3, 74.0)
- turned S1 to 0 degrees
- turned S2 to 180 degrees
- renumbered REF** to SWITCH
Connections:
- 0 pad 1: (no net) -> GND
- BQ24075 pad CHG_N: VDDH -> CHG
- Button pad 2: (no net) -> RST
- Button pad 3: (no net) -> GND
- Button pad 4: (no net) -> GND
- E73 pad 10 P0.30: K4 -> K10
- E73 pad 14 P0.06: (no net) -> K13
- E73 pad 15 P0.05: (no net) -> K1
- E73 pad 16 P0.08: (no net) -> K8
- E73 pad 17 P1.09: (no net) -> K2
- E73 pad 18 P0.04: (no net) -> K14
- E73 pad 20 P0.12: (no net) -> K9
- E73 pad 22 P0.07: (no net) -> K15
- E73 pad 26 RST: (no net) -> RST
- E73 pad 28 P0.15: (no net) -> K7
- E73 pad 30 P0.17: (no net) -> K16
- E73 pad 32 P0.20: (no net) -> STATUS
- E73 pad 33 P0.13: (no net) -> K17
- E73 pad 35 P0.24: (no net) -> K19
- E73 pad 37 SWDIO: (no net) -> SWIO
- E73 pad 39 SWDCLK: (no net) -> SWCLK
- E73 pad 41 P0.09: (no net) -> K20
- E73 pad 43 P0.10: (no net) -> K21
- E73 pad 9 P0.31: K17 -> K4
- JST pad 1: GND -> VBAT
- JST pad 2: VBAT -> GND
- JST pad S1: (no net) -> GND
- JST pad S2: (no net) -> GND
- REF** pad 1: (no net) -> GND (x4)
- SWITCH pad S1: (no net) -> GND
- SWITCH pad S2: (no net) -> GND
- SWITCH pad S3: (no net) -> GND
- SWITCH pad S4: (no net) -> GND
Routing:
- net VBUS: track 24.5 -> 128.2 mm, vias 1 -> 2
- net RST: track 0.00 -> 73.5 mm, vias 0 -> 2
- net CHG: track 0.00 -> 52.2 mm, vias 0 -> 2
- net VDDH: track 24.0 -> 73.1 mm
- net K19: track 0.00 -> 36.3 mm
- net K16: track 14.5 -> 50.4 mm, vias 0 -> 2
- net K10: track 24.4 -> 55.8 mm
- net SWCLK: track 0.00 -> 27.5 mm, vias 0 -> 1
- net D-: track 30.7 -> 56.0 mm, vias 2 -> 3
- net D+: track 31.0 -> 54.7 mm, vias 1 -> 2
- net K7: track 103.9 -> 125.9 mm
- net SWIO: track 0.00 -> 21.4 mm, vias 0 -> 1
- net STATUS: track 0.00 -> 20.8 mm, vias 0 -> 2
- net K20: track 0.00 -> 19.8 mm
- net K14: track 102.8 -> 122.2 mm, vias 0 -> 2
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