File: V0.2/main.kicad_sch (KiCad schematic)
At the start: 42 parts, among them J1 Conn_01x02_Female, J1 USB_C_2.0, SW1 SW_DPST_x2, SW10 SW_DPST_x2, SW11 SW_DPST_x2, SW12 SW_DPST_x2, SW13 SW_DPST_x2, SW14 SW_DPST_x2, SW15 SW_DPST_x2, SW16 SW_DPST_x2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

Commit message: Finalized design
Parts:
- removed F1: Polyfuse, symbol Device:Polyfuse
- D1: value (none) -> RED LED
- D2: value (none) -> BLUE LED
- R6: value (none) -> 1kΩ
- U1: value (none) -> E73-2G4M08S1E
- U2: value BQ24075 -> (none); footprint Package_DFN_QFN:VQFN-16-1EP_3x3mm_P0.5mm_EP1.6x1.6mm -> (none)
Connections:
- net GND: now also J1.S1 (SHIELD)
- net VBUS: now also J1.A4 (VBUS), J1.A9 (VBUS), J1.B4 (VBUS), J1.B9 (VBUS)
- no-connect marks 9 -> 8
Other:
- moved on the sheet: R1, R2
