File: V0.3/Choc/main.kicad_sch (KiCad schematic)
At the start: 80 parts, among them J1 USB_C_2.0, J2 JST-BAT, J3 SWD, J4 USB_C_2.0, J5 JST-BAT, J6 SWD, SW10 SW_DPST_x2, SW11 SW_DPST_x2, SW12 SW_DPST_x2, SW13 SW_DPST_x2, SW14 SW_DPST_x2, SW15 SW_DPST_x2, SW16 SW_DPST_x2, SW17 SW_DPST_x2, SW18 SW_DPST_x2, SW19 SW_DPST_x2, SW2 SW_DPST_x2, SW20 SW_DPST_x2, SW21 SW_DPST_x2, SW22 SW_DPST_x2, SW23 SW_DPST_x2, SW24 SW_DPST_x2, SW25 SW_DPST_x2, SW26 SW_DPST_x2, SW27 SW_DPST_x2, SW28 SW_DPST_x2, SW29 SW_DPST_x2, SW3 SW_DPST_x2, SW30 SW_DPST_x2, SW31 SW_DPST_x2, SW32 SW_DPST_x2, SW33 SW_DPST_x2, SW34 SW_DPST_x2, SW35 SW_DPST_x2, SW36 SW_DPST_x2, SW37 SW_DPST_x2, SW38 SW_DPST_x2, SW39 SW_DPST_x2, SW4 SW_DPST_x2, SW40 SW_DPST_x2, SW41 SW_DPST_x2, SW42 SW_DPST_x2, SW5 SW_DPST_x2, SW6 SW_DPST_x2, SW7 SW_DPST_x2, SW8 SW_DPST_x2, SW9 SW_DPST_x2, U1 MS88SF31_Min, U2 BQ24072, U3 IP4234CZ6, U4 MS88SF31_Min, U5 BQ24072, U6 IP4234CZ6

Commit message: V0.4
Parts:
- SW1: value (none) -> SW_DPST_x2
Connections:
- net VDDH: now also U1.31 (VDD), U4.31 (VDD)
- no-connect marks 51 -> 49
Other:
- title: Contour Split -> Gravi
Changed lines of the file:
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@@
   (paper "User" 340.004 240.005)
   (title_block
-    (title "Contour Split")
+    (title "Gravi")
     (date "2023-01-16")
     (rev "3")
@@
   (no_connect (at 176.53 43.18))
   (no_connect (at 283.21 50.8))
-  (no_connect (at 189.23 73.66))
   (no_connect (at 39.37 114.3))
   (no_connect (at 184.15 73.66))
@@
   (no_connect (at 24.13 30.48))
   (no_connect (at 74.93 25.4))
-  (no_connect (at 36.83 73.66))
   (no_connect (at 31.75 73.66))
   (no_connect (at 24.13 43.18))
@@
     (stroke (width 0) (type default) (color 0 0 0 0))
   )
+  (wire (pts (xy 186.69 73.66) (xy 189.23 73.66))
+    (stroke (width 0) (type default) (color 0 0 0 0))
+  )
   (wire (pts (xy 20.32 158.75) (xy 22.86 158.75))
     (stroke (width 0) (type default) (color 0 0 0 0))
@@
   )
   (wire (pts (xy 193.04 153.67) (xy 184.15 153.67))
+    (stroke (width 0) (type default) (color 0 0 0 0))
+  )
+  (wire (pts (xy 34.29 73.66) (xy 36.83 73.66))
     (stroke (width 0) (type default) (color 0 0 0 0))
   )
@@
     )
   )
-  (global_label "VDDH" (shape input) (at 34.29 73.66 270) (fields_autoplaced)
-    (effects (font (size 1.27 1.27)) (justify right))
-    (property "Intersheet References" "${INTERSHEET_REFS}" (id 0) (at 34.2106 81.0321 90)
+  (global_label "VDDH" (shape input) (at 35.56 73.66 270) (fields_autoplaced)
+    (effects (font (size 1.27 1.27)) (justify right))
+    (property "Intersheet References" "${INTERSHEET_REFS}" (id 0) (at 35.4806 81.0321 90)
       (effects (font (size 1.27 1.27)) (justify right) hide)
     )
@@
     )
   )
-  (global_label "VDDH" (shape input) (at 186.69 73.66 270) (fields_autoplaced)
-    (effects (font (size 1.27 1.27)) (justify right))
-    (property "Intersheet References" "${INTERSHEET_REFS}" (id 0) (at 186.6106 81.0321 90)
+  (global_label "VDDH" (shape input) (at 187.96 73.66 270) (fields_autoplaced)
+    (effects (font (size 1.27 1.27)) (justify right))
+    (property "Intersheet References" "${INTERSHEET_REFS}" (id 0) (at 187.8806 81.0321 90)
       (effects (font (size 1.27 1.27)) (justify right) hide)
     )
@@
     (in_bom yes) (on_board yes)
     (property "Reference" "SW1" (id 0) (at 22.86 127 0))
-    (property "Value" "" (id 1) (at 36.83 127 0))
+    (property "Value" "SW_DPST_x2" (id 1) (at 36.83 127 0))
     (property "Footprint" "" (id 2) (at 27.94 128.27 0)
       (effects (font (size 1.27 1.27)) hide)
